Commit message: Give modified dual bolt package a unique ROS name

File: sim_ws/src/fr3_dual_bolt_cell_modified/urdf/common.urdf.xacro (robot description, xacro)
@@ -2,5 +2,5 @@
 <robot name="fairino3_v6_robot" xmlns:xacro="http://www.ros.org/wiki/xacro">
   <!-- Explicit paths also allow non-ROS offline Xacro tests. -->
-  <xacro:arg name="scene_file" default="$(find fr3_dual_bolt_cell)/config/scene.yaml"/>
+  <xacro:arg name="scene_file" default="$(find fr3_dual_bolt_cell_modified)/config/scene.yaml"/>
   <xacro:property name="scene" value="${xacro.load_yaml('$(arg scene_file)')}"/>
   <xacro:property name="support" value="${scene['support']}"/>

File: sim_ws/src/fr3_dual_bolt_cell_modified/urdf/fr3_arm.urdf (robot description, URDF)
Before this commit: robot fairino3_v6_robot, 7 links, 6 joints
Links:
- link base_link: geometry collision mesh filename=package://fr3_dual_bolt_cell_modified/meshes/fairino3_v6/ba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; visual mesh filename=package://fr3_dual_bolt_cell_modified/meshes/fairino3_v6/ba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
- link forearm_link: geometry collision mesh filename=package://fr3_dual_bolt_cell_modified/meshes/fairino3_v6/fo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; visual mesh filename=package://fr3_dual_bolt_cell_modified/meshes/fairino3_v6/fo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
- link shoulder_link: geometry collision mesh filename=package://fr3_dual_bolt_cell_modified/meshes/fairino3_v6/sh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; visual mesh filename=package://fr3_dual_bolt_cell_modified/meshes/fairino3_v6/sh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
- link upperarm_link: geometry collision mesh filename=package://fr3_dual_bolt_cell_modified/meshes/fairino3_v6/up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; visual mesh filename=package://fr3_dual_bolt_cell_modified/meshes/fairino3_v6/up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
- link wrist1_link: geometry collision mesh filename=package://fr3_dual_bolt_cell_modified/meshes/fairino3_v6/wr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; visual mesh filename=package://fr3_dual_bolt_cell_modified/meshes/fairino3_v6/wr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
- link wrist2_link: geometry collision mesh filename=package://fr3_dual_bolt_cell_modified/meshes/fairino3_v6/wr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; visual mesh filename=package://fr3_dual_bolt_cell_modified/meshes/fairino3_v6/wr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
- link wrist3_link: geometry collision mesh filename=package://fr3_dual_bolt_cell_modified/meshes/fairino3_v6/wr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; visual mesh filename=package://fr3_dual_bolt_cell_modified/meshes/fairino3_v6/wr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
